File: discipline-pcb.kicad_pcb (KiCad board)
At the start: 2 copper layers, 304.9 x 122.8 mm, 180 parts, among them J1 AVR-ISP-6, SW1 KEYSW, SW10 KEYSW, SW11 KEYSW, SW12 KEYSW, SW13 KEYSW, SW14 KEYSW, SW15 KEYSW, SW16 KEYSW, SW17 KEYSW, SW18 KEYSW, SW19 KEYSW, SW2 KEYSW, SW20 KEYSW, SW21 KEYSW, SW22 KEYSW, SW23 KEYSW, SW24 KEYSW, SW25 KEYSW, SW26 KEYSW, SW27 KEYSW, SW28 KEYSW, SW29 KEYSW, SW3 KEYSW, SW30 KEYSW, SW31 KEYSW, SW32 KEYSW, SW33 KEYSW, SW34 KEYSW, SW35 KEYSW, SW36 KEYSW, SW37 KEYSW, SW38 KEYSW, SW39 KEYSW, SW4 KEYSW, SW40 KEYSW, SW41 KEYSW, SW42 KEYSW, SW43 KEYSW, SW44 KEYSW, SW45 KEYSW, SW46 KEYSW, SW47 KEYSW, SW48 KEYSW, SW49 KEYSW, SW5 KEYSW, SW50 KEYSW, SW51 KEYSW, SW52 KEYSW, SW53 KEYSW, SW54 KEYSW, SW55 KEYSW, SW56 KEYSW, SW57 KEYSW, SW58 KEYSW, SW59 KEYSW, SW6 KEYSW, SW60 KEYSW, SW61 KEYSW, SW62 KEYSW, SW63 KEYSW, SW64 KEYSW, SW65 KEYSW, SW66 KEYSW, SW67 KEYSW, SW68 KEYSW, SW69 KEYSW, SW7 KEYSW, SW70 KEYSW, SW71 KEYSW, SW72 KEYSW, SW73 KEYSW, SW74 KEYSW, SW8 KEYSW, SW9 KEYSW, U1 ATmega32A-PU, Y1 Crystal

Commit message: Initial hotswap version
Parts:
- removed the G*** at (354.1, 71.1)
- removed the G*** at (58.5, 71.1)
- removed the G*** at (155.2, 163.6) (x2)
- removed REF**: 6.25U, cftkb:MX-6.25U-Stabilizer
- removed REF** (x10): MountingHole_2.2mm_M2_Pad, MountingHole:MountingHole_2.2mm_M2_Pad
- removed ST72: 7U, cftkb:MX-7U-Stabilizer
- removed SW71, SW73, SW74: KEYSW, cftkb:SW_Cherry_MX1A_1.50u_PCBNOSCREEN
- removed SW72: KEYSW, cftkb:SW_Cherry_MX1A_1.00u_PCB-NOSCREEN
- added G***: LOGO, logos:TOPY 4MM MASK, F.Cu at (44.3, 49.3)
- added G***: LOGO, logos:TOPY 4MM MASK, F.Cu at (339.9, 49.3)
- added H1: MountingHole_2.2mm_M2_Pad_Via, MountingHole:MountingHole_2.2mm_M2_Pad_Via, F.Cu at (44.3, 40.1)
- added H10: MountingHole_2.2mm_M2_Pad_Via, MountingHole:MountingHole_2.2mm_M2_Pad_Via, F.Cu at (301.7, 139.4)
- added H2: MountingHole_2.2mm_M2_Pad_Via, MountingHole:MountingHole_2.2mm_M2_Pad_Via, F.Cu at (44.3, 58.5)
- added H3: MountingHole_2.2mm_M2_Pad_Via, MountingHole:MountingHole_2.2mm_M2_Pad_Via, F.Cu at (339.8, 40.1)
- added H4: MountingHole_2.2mm_M2_Pad_Via, MountingHole:MountingHole_2.2mm_M2_Pad_Via, F.Cu at (339.8, 58.5)
- added H5: MountingHole_2.2mm_M2_Pad_Via, MountingHole:MountingHole_2.2mm_M2_Pad_Via, F.Cu at (99.6, 82.5)
- added H6: MountingHole_2.2mm_M2_Pad_Via, MountingHole:MountingHole_2.2mm_M2_Pad_Via, F.Cu at (192.1, 82.5)
- added H7: MountingHole_2.2mm_M2_Pad_Via, MountingHole:MountingHole_2.2mm_M2_Pad_Via, F.Cu at (284.5, 82.5)
- added H8: MountingHole_2.2mm_M2_Pad_Via, MountingHole:MountingHole_2.2mm_M2_Pad_Via, F.Cu at (82.4, 139.4)
- added H9: MountingHole_2.2mm_M2_Pad_Via, MountingHole:MountingHole_2.2mm_M2_Pad_Via, F.Cu at (192.1, 145.2)
- SW1, SW10, SW11, SW12, SW13, SW15, SW17, SW18, SW19, SW2, SW20, SW21, SW22, SW23, SW24, SW25, SW26, SW27, SW28, SW3, SW30, SW32, SW33, SW34, SW35, SW36, SW37, SW38, SW39, SW4, SW40, SW41, SW42, SW44, SW46, SW47, SW48, SW49, SW5, SW50, SW51, SW52, SW53, SW54, SW55, SW57, SW58, SW6, SW65, SW66, SW67, SW68, SW7, SW8, SW9: footprint cftkb:SW_Cherry_MX1A_1.00u_PCB-NOSCREEN -> MX_Only:MXOnly-1U-Hotswap
- SW14: footprint cftkb:SW_Cherry_MX1A_2.00u_PCBNOSCREEN -> MX_Only:MXOnly-2U-Hotswap
- SW16, SW29: footprint cftkb:SW_Cherry_MX1A_1.50u_PCBNOSCREEN -> MX_Only:MXOnly-1.5U-Hotswap
- SW31, SW56: footprint cftkb:SW_Cherry_MX1A_1.75u_PCBNOSCREEN -> MX_Only:MXOnly-1.75U-Hotswap
- SW43, SW45: footprint cftkb:SW_Cherry_MX1A_2.25u_PCBNOSCREEN -> MX_Only:MXOnly-2.25U-Hotswap
- SW59, SW61, SW69: footprint cftkb:SW_Cherry_MX1A_1.25u_PCBNOSCREEN -> MX_Only:MXOnly-1.25U-Hotswap
- SW60: footprint cftkb:SW_Cherry_MX1A_1.25u_PCBNOSCREEN -> MX_Only:MXOnly-1U-Hotswap
- SW62: footprint cftkb:SW_Cherry_MX1A_1.00u_PCB-NOSCREEN -> MX_Only:MXOnly-7U-Hotswap-ReversedStabilizers
- SW63, SW64: footprint cftkb:SW_Cherry_MX1A_1.00u_PCB-NOSCREEN -> MX_Only:MXOnly-1.25U-Hotswap
- SW70: footprint cftkb:SW_Cherry_MX1A_1.50u_PCBNOSCREEN -> MX_Only:MXOnly-1U-Hotswap
- moved SW70 244.5 mm to (296.8, 73.0), turned to 180 degrees
- moved SW68 95.3 mm to (315.9, 73.0), turned to 180 degrees
- moved D43 38.0 mm to (204.8, 46.1)
- moved D48 35.7 mm to (100.2, 44.5)
- moved D53 35.7 mm to (163.6, 44.5)
- moved D54 35.7 mm to (176.2, 44.5)
- moved D55 35.7 mm to (188.9, 44.5)
- moved D46 35.7 mm to (74.8, 44.5)
- moved D47 35.7 mm to (87.5, 44.5)
- moved D49 35.7 mm to (112.9, 44.5)
- moved D50 35.7 mm to (125.5, 44.5)
- moved D51 35.7 mm to (138.2, 44.5)
- moved D52 35.7 mm to (150.9, 44.5)
- moved D57 35.6 mm to (214.2, 44.5)
- moved D68 34.4 mm to (220.5, 47.8)
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Connections:
- D29 pad 1: row1 -> row2
- D68 pad 1: row4 -> row1
- SW1 pad 1: col0 -> Net-(D1-Pad2)
- SW1 pad 2: Net-(D1-Pad2) -> col0
- SW10 pad 1: col9 -> Net-(D10-Pad2)
- SW10 pad 2: Net-(D10-Pad2) -> col9
- SW11 pad 1: col10 -> Net-(D11-Pad2)
- SW11 pad 2: Net-(D11-Pad2) -> col10
- SW12 pad 1: col11 -> Net-(D12-Pad2)
- SW12 pad 2: Net-(D12-Pad2) -> col11
- SW13 pad 1: col12 -> Net-(D13-Pad2)
- SW13 pad 2: Net-(D13-Pad2) -> col12
- SW14 pad 1: col13 -> Net-(D14-Pad2)
- SW14 pad 2: Net-(D14-Pad2) -> col13
- SW15 pad 1: col14 -> Net-(D15-Pad2)
- SW15 pad 2: Net-(D15-Pad2) -> col14
- SW16 pad 1: col0 -> Net-(D16-Pad2)
- SW16 pad 2: Net-(D16-Pad2) -> col0
- SW17 pad 1: col1 -> Net-(D17-Pad2)
- SW17 pad 2: Net-(D17-Pad2) -> col1
- SW18 pad 1: col2 -> Net-(D18-Pad2)
- SW18 pad 2: Net-(D18-Pad2) -> col2
- SW19 pad 1: col3 -> Net-(D19-Pad2)
- SW19 pad 2: Net-(D19-Pad2) -> col3
- SW2 pad 1: col1 -> Net-(D2-Pad2)
- SW2 pad 2: Net-(D2-Pad2) -> col1
- SW20 pad 1: col4 -> Net-(D20-Pad2)
- SW20 pad 2: Net-(D20-Pad2) -> col4
- SW21 pad 1: col5 -> Net-(D21-Pad2)
- SW21 pad 2: Net-(D21-Pad2) -> col5
- SW22 pad 1: col6 -> Net-(D22-Pad2)
- SW22 pad 2: Net-(D22-Pad2) -> col6
- SW23 pad 1: col7 -> Net-(D23-Pad2)
- SW23 pad 2: Net-(D23-Pad2) -> col7
- SW24 pad 1: col8 -> Net-(D24-Pad2)
- SW24 pad 2: Net-(D24-Pad2) -> col8
- SW25 pad 1: col9 -> Net-(D25-Pad2)
- SW25 pad 2: Net-(D25-Pad2) -> col9
- SW26 pad 1: col10 -> Net-(D26-Pad2)
- SW26 pad 2: Net-(D26-Pad2) -> col10
- SW27 pad 1: col11 -> Net-(D27-Pad2)
- SW27 pad 2: Net-(D27-Pad2) -> col11
- SW28 pad 1: col12 -> Net-(D28-Pad2)
- SW28 pad 2: Net-(D28-Pad2) -> col12
- SW29 pad 1: col13 -> Net-(D29-Pad2)
- SW29 pad 2: Net-(D29-Pad2) -> col13
- SW3 pad 1: col2 -> Net-(D3-Pad2)
- SW3 pad 2: Net-(D3-Pad2) -> col2
- SW30 pad 1: col14 -> Net-(D30-Pad2)
- SW30 pad 2: Net-(D30-Pad2) -> col14
- SW32 pad 1: col1 -> Net-(D32-Pad2)
- SW32 pad 2: Net-(D32-Pad2) -> col1
- SW33 pad 1: col2 -> Net-(D33-Pad2)
- SW33 pad 2: Net-(D33-Pad2) -> col2
- SW34 pad 1: col3 -> Net-(D34-Pad2)
- SW34 pad 2: Net-(D34-Pad2) -> col3
- SW35 pad 1: col4 -> Net-(D35-Pad2)
- SW35 pad 2: Net-(D35-Pad2) -> col4
- SW36 pad 1: col5 -> Net-(D36-Pad2)
- SW36 pad 2: Net-(D36-Pad2) -> col5
- SW37 pad 1: col6 -> Net-(D37-Pad2)
- SW37 pad 2: Net-(D37-Pad2) -> col6
- SW38 pad 1: col7 -> Net-(D38-Pad2)
- SW38 pad 2: Net-(D38-Pad2) -> col7
- SW39 pad 1: col8 -> Net-(D39-Pad2)
- SW39 pad 2: Net-(D39-Pad2) -> col8
- SW4 pad 1: col3 -> Net-(D4-Pad2)
- SW4 pad 2: Net-(D4-Pad2) -> col3
- SW40 pad 1: col9 -> Net-(D40-Pad2)
- SW40 pad 2: Net-(D40-Pad2) -> col9
- SW41 pad 1: col10 -> Net-(D41-Pad2)
- SW41 pad 2: Net-(D41-Pad2) -> col10
- SW42 pad 1: col11 -> Net-(D42-Pad2)
- SW42 pad 2: Net-(D42-Pad2) -> col11
- SW43 pad 1: col13 -> Net-(D43-Pad2)
- SW43 pad 2: Net-(D43-Pad2) -> col12
- SW44 pad 1: col14 -> Net-(D44-Pad2)
- SW44 pad 2: Net-(D44-Pad2) -> col14
- SW45 pad 1: col0 -> Net-(D45-Pad2)
- SW45 pad 2: Net-(D45-Pad2) -> col0
- SW46 pad 1: col2 -> Net-(D46-Pad2)
- SW46 pad 2: Net-(D46-Pad2) -> col2
- SW47 pad 1: col3 -> Net-(D47-Pad2)
- SW47 pad 2: Net-(D47-Pad2) -> col3
- SW48 pad 1: col4 -> Net-(D48-Pad2)
- SW48 pad 2: Net-(D48-Pad2) -> col4
- SW49 pad 1: col5 -> Net-(D49-Pad2)
- SW49 pad 2: Net-(D49-Pad2) -> col5
- SW5 pad 1: col4 -> Net-(D5-Pad2)
- SW5 pad 2: Net-(D5-Pad2) -> col4
- SW50 pad 1: col6 -> Net-(D50-Pad2)
- SW50 pad 2: Net-(D50-Pad2) -> col6
- SW51 pad 1: col7 -> Net-(D51-Pad2)
- SW51 pad 2: Net-(D51-Pad2) -> col7
- SW52 pad 1: col8 -> Net-(D52-Pad2)
- SW52 pad 2: Net-(D52-Pad2) -> col8
- SW53 pad 1: col9 -> Net-(D53-Pad2)
- SW53 pad 2: Net-(D53-Pad2) -> col9
- SW54 pad 1: col10 -> Net-(D54-Pad2)
- SW54 pad 2: Net-(D54-Pad2) -> col10
- SW55 pad 1: col11 -> Net-(D55-Pad2)
- SW55 pad 2: Net-(D55-Pad2) -> col11
- SW56 pad 1: col12 -> Net-(D56-Pad2)
- SW56 pad 2: Net-(D56-Pad2) -> col12
- SW57 pad 1: col13 -> Net-(D57-Pad2)
- SW57 pad 2: Net-(D57-Pad2) -> col13
- SW58 pad 1: col14 -> Net-(D58-Pad2)
- SW58 pad 2: Net-(D58-Pad2) -> col14
- SW59 pad 1: col0 -> Net-(D59-Pad2)
- SW59 pad 2: Net-(D59-Pad2) -> col0
- SW6 pad 1: col5 -> Net-(D6-Pad2)
- SW6 pad 2: Net-(D6-Pad2) -> col5
- SW60 pad 1: col1 -> Net-(D60-Pad2)
- SW60 pad 2: Net-(D60-Pad2) -> col1
- SW61 pad 1: col2 -> Net-(D61-Pad2)
- SW61 pad 2: Net-(D61-Pad2) -> col2
- SW62 pad 1: col6 -> Net-(D62-Pad2)
- SW62 pad 2: Net-(D62-Pad2) -> col6
- SW63 pad 1: col9 -> Net-(D63-Pad2)
- SW63 pad 2: Net-(D63-Pad2) -> col10
- SW64 pad 1: col10 -> Net-(D64-Pad2)
- SW64 pad 2: Net-(D64-Pad2) -> col11
- SW65 pad 1: col12 -> Net-(D65-Pad2)
- SW65 pad 2: Net-(D65-Pad2) -> col12
- SW66 pad 1: col13 -> Net-(D66-Pad2)
- SW66 pad 2: Net-(D66-Pad2) -> col13
- SW67 pad 1: col14 -> Net-(D67-Pad2)
- SW67 pad 2: Net-(D67-Pad2) -> col14
- SW68 pad 1: col11 -> col13
- SW69 pad 1: col0 -> Net-(D31-Pad2)
- SW69 pad 2: Net-(D31-Pad2) -> col0
- SW7 pad 1: col6 -> Net-(D7-Pad2)
- SW7 pad 2: Net-(D7-Pad2) -> col6
- SW70 pad 1: col0 -> col13
- SW70 pad 2: Net-(D59-Pad2) -> Net-(D14-Pad2)
- SW8 pad 1: col7 -> Net-(D8-Pad2)
- SW8 pad 2: Net-(D8-Pad2) -> col7
- SW9 pad 1: col8 -> Net-(D9-Pad2)
- SW9 pad 2: Net-(D9-Pad2) -> col8
Routing:
- net Net-(D68-Pad2): track 232.5 -> 109.9 mm, vias 0 -> 1
- net Net-(D64-Pad2): track 187.5 -> 238.5 mm, vias 0 -> 1
- net col9: track 260.1 -> 214.9 mm
- net col10: track 251.0 -> 219.8 mm
- net row3: track 287.2 -> 259.2 mm, vias 3 -> 1
- net Net-(D63-Pad2): track 279.4 -> 260.1 mm, vias 0 -> 1
- net row4: track 296.4 -> 277.4 mm
- net col2: track 329.2 -> 310.4 mm
- net Net-(D62-Pad2): track 355.8 -> 338.6 mm, vias 0 -> 1
- net Net-(D13-Pad2): track 82.3 -> 66.8 mm, vias 0 -> 1
- net col6: track 279.4 -> 264.2 mm
- net Net-(D43-Pad2): track 140.6 -> 125.7 mm, vias 0 -> 1
- net Net-(D12-Pad2): track 76.4 -> 61.8 mm, vias 0 -> 1
- net col7: track 269.9 -> 255.4 mm
- net Net-(D11-Pad2): track 69.9 -> 55.8 mm, vias 0 -> 1
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Other:
- board text added: "1.0.0"
- board text added: "21/03/2020"
- board text added: "DISCIPLINE - HS Hotswap (kailh sockets) version of DISCIPLINE"
- board text added: "DISCIPLINE-HS"
- board text added: "Derived from DISCIPLINE rev1 coseyfannitutti 2019"
- board text added: "nsmk rev1.0.0"
- board text removed: "1"
- board text removed: "1.25U"
- board text removed: "1.5U"
- board text removed: "1U"
- board text removed: "7/2/2019"
- board text removed: "DISCIPLINE - 65% keyboard made with only through hole components"
- board text removed: "STANDARD"
- board text removed: "STEPPED"
- board text removed: "coseyfannitutti 2019 rev1"
