File: discipline-pcb.kicad_pcb (KiCad board)
At the start: 2 copper layers, 304.9 x 122.8 mm, 172 parts, among them J1 AVR-ISP-6, SW1 KEYSW, SW10 KEYSW, SW11 KEYSW, SW12 KEYSW, SW13 KEYSW, SW14 KEYSW, SW15 KEYSW, SW16 KEYSW, SW17 KEYSW, SW18 KEYSW, SW19 KEYSW, SW2 KEYSW, SW20 KEYSW, SW21 KEYSW, SW22 KEYSW, SW23 KEYSW, SW24 KEYSW, SW25 KEYSW, SW26 KEYSW, SW27 KEYSW, SW28 KEYSW, SW29 KEYSW, SW3 KEYSW, SW30 KEYSW, SW31 KEYSW, SW32 KEYSW, SW33 KEYSW, SW34 KEYSW, SW35 KEYSW, SW36 KEYSW, SW37 KEYSW, SW38 KEYSW, SW39 KEYSW, SW4 KEYSW, SW40 KEYSW, SW41 KEYSW, SW42 KEYSW, SW43 KEYSW, SW44 KEYSW, SW45 KEYSW, SW46 KEYSW, SW47 KEYSW, SW48 KEYSW, SW49 KEYSW, SW5 KEYSW, SW50 KEYSW, SW51 KEYSW, SW52 KEYSW, SW53 KEYSW, SW54 KEYSW, SW55 KEYSW, SW56 KEYSW, SW57 KEYSW, SW58 KEYSW, SW59 KEYSW, SW6 KEYSW, SW60 KEYSW, SW61 KEYSW, SW62 KEYSW, SW63 KEYSW, SW64 KEYSW, SW65 KEYSW, SW66 KEYSW, SW67 KEYSW, SW68 KEYSW, SW69 KEYSW, SW7 KEYSW, SW70 KEYSW, SW8 KEYSW, SW9 KEYSW, U1 ATmega32A-PU, Y1 Crystal

Commit message: Add alternative bottom row
Parts:
- added SW71: KEYSW, MX_Only:MXOnly-7U-Hotswap, F.Cu at (173.0, 149.2)
- added SW72: KEYSW, MX_Only:MXOnly-1.25U-Hotswap, F.Cu at (251.6, 149.2)
- added SW73: KEYSW, MX_Only:MXOnly-1.25U-Hotswap, F.Cu at (275.4, 149.2)
- added SW74: KEYSW, MX_Only:MXOnly-1U-Hotswap, F.Cu at (73.0, 149.2)
- added SW75: KEYSW, MX_Only:MXOnly-1.25U-Hotswap, F.Cu at (94.5, 149.2)
- H1, H10, H2, H3, H4, H5, H6, H7, H8, H9: value MountingHole_2.2mm_M2_Pad_Via -> MountingHole_Pad
- SW60: footprint MX_Only:MXOnly-1U-Hotswap -> MX_Only:MXOnly-1.25U-Hotswap
- SW62: footprint MX_Only:MXOnly-7U-Hotswap-ReversedStabilizers -> MX_Only:MXOnly-6.25U-Hotswap-ReversedStabilizers
- SW63, SW64: footprint MX_Only:MXOnly-1.25U-Hotswap -> MX_Only:MXOnly-1.5U-Hotswap
- moved SW63 7.14 mm to (244.5, 149.2)
- moved SW61 4.76 mm to (99.2, 149.2)
- moved SW60 2.38 mm to (75.4, 149.2)
- moved SW62 2.38 mm to (170.6, 149.2)
- moved SW64 2.38 mm to (273.0, 149.2)
Connections:
- H1 pad 1: (no net) -> Net-(H1-Pad1)
- H10 pad 1: (no net) -> Net-(H10-Pad1)
- H2 pad 1: (no net) -> Net-(H2-Pad1)
- H3 pad 1: (no net) -> Net-(H3-Pad1)
- H4 pad 1: (no net) -> Net-(H4-Pad1)
- H5 pad 1: (no net) -> Net-(H5-Pad1)
- H6 pad 1: (no net) -> Net-(H6-Pad1)
- H7 pad 1: (no net) -> Net-(H7-Pad1)
- H8 pad 1: (no net) -> Net-(H8-Pad1)
- H9 pad 1: (no net) -> Net-(H9-Pad1)
Routing:
- net Net-(D61-Pad2): track 415.3 -> 429.9 mm
- net Net-(D63-Pad2): track 260.1 -> 272.4 mm
- net col10: track 219.8 -> 231.3 mm
- net Net-(D64-Pad2): track 238.5 -> 249.8 mm
- net Net-(D62-Pad2): track 338.6 -> 349.8 mm
- net col2: track 310.4 -> 321.5 mm
- net Net-(D59-Pad2): track 455.2 -> 465.3 mm
- net col1: track 311.6 -> 321.1 mm
- net Net-(D60-Pad2): track 101.6 -> 110.7 mm
- net col11: track 201.0 -> 209.2 mm
- net col6: track 264.2 -> 272.4 mm
- net Net-(D65-Pad2): track 219.3 -> 225.5 mm
- net GND: vias 35 -> 30
- net (no net): vias 2 -> 1
Other:
- board text added: "nsmk rev1.1.0"
- board text removed: "nsmk rev1.0.0"
