File: discipline-pcb.sch (KiCad schematic (older format))
At the start: 164 parts, among them J1 AVR-ISP-6, SW1 KEYSW, SW10 KEYSW, SW11 KEYSW, SW12 KEYSW, SW13 KEYSW, SW14 KEYSW, SW15 KEYSW, SW16 KEYSW, SW17 KEYSW, SW18 KEYSW, SW19 KEYSW, SW2 KEYSW, SW20 KEYSW, SW21 KEYSW, SW22 KEYSW, SW23 KEYSW, SW24 KEYSW, SW25 KEYSW, SW26 KEYSW, SW27 KEYSW, SW28 KEYSW, SW29 KEYSW, SW3 KEYSW, SW30 KEYSW, SW31 KEYSW, SW32 KEYSW, SW33 KEYSW, SW34 KEYSW, SW35 KEYSW, SW36 KEYSW, SW37 KEYSW, SW38 KEYSW, SW39 KEYSW, SW4 KEYSW, SW40 KEYSW, SW41 KEYSW, SW42 KEYSW, SW43 KEYSW, SW44 KEYSW, SW45 KEYSW, SW46 KEYSW, SW47 KEYSW, SW48 KEYSW, SW49 KEYSW, SW5 KEYSW, SW50 KEYSW, SW51 KEYSW, SW52 KEYSW, SW53 KEYSW, SW54 KEYSW, SW55 KEYSW, SW56 KEYSW, SW57 KEYSW, SW58 KEYSW, SW59 KEYSW, SW6 KEYSW, SW60 KEYSW, SW61 KEYSW, SW62 KEYSW, SW63 KEYSW, SW64 KEYSW, SW65 KEYSW, SW66 KEYSW, SW67 KEYSW, SW68 KEYSW, SW69 KEYSW, SW7 KEYSW, SW70 KEYSW, SW71 KEYSW, SW72 KEYSW, SW73 KEYSW, SW74 KEYSW, SW8 KEYSW, SW9 KEYSW, U1 ATmega32A-PU, Y1 Crystal

Commit message: Initial hotswap version
Parts:
- removed SW70, SW71, SW73, SW74: KEYSW, cftkb:SW_Cherry_MX1A_1.50u_PCBNOSCREEN, symbol keyboard_parts:KEYSW
- removed SW72: KEYSW, cftkb:SW_Cherry_MX1A_1.00u_PCB-NOSCREEN, symbol keyboard_parts:KEYSW
- added H1, H10, H2, H3, H4, H5, H6, H7, H8, H9: MountingHole_Pad, MountingHole:MountingHole_2.2mm_M2_Pad_Via, symbol Mechanical:MountingHole_Pad
- added SW68: KEYSW, MX_Only:MXOnly-1U-Hotswap, symbol discipline-pcb-rescue:KEYSW-keyboard_parts
- BOOT1, RESET1: symbol keyboard_parts:SW_PUSH -> discipline-pcb-rescue:SW_PUSH-keyboard_parts
- J1: symbol Connector:AVR-ISP-6 -> discipline-pcb-rescue:AVR-ISP-6-Connector
- SW1, SW10, SW11, SW12, SW13, SW15, SW17, SW18, SW19, SW2, SW20, SW21, SW22, SW23, SW24, SW25, SW26, SW27, SW28, SW3, SW30, SW32, SW33, SW34, SW35, SW36, SW37, SW38, SW39, SW4, SW40, SW41, SW42, SW44, SW46, SW47, SW48, SW49, SW5, SW50, SW51, SW52, SW53, SW54, SW55, SW57, SW58, SW6, SW65, SW66, SW67, SW7, SW8, SW9: footprint cftkb:SW_Cherry_MX1A_1.00u_PCB-NOSCREEN -> MX_Only:MXOnly-1U-Hotswap; symbol keyboard_parts:KEYSW -> discipline-pcb-rescue:KEYSW-keyboard_parts
- SW14: footprint cftkb:SW_Cherry_MX1A_2.00u_PCBNOSCREEN -> MX_Only:MXOnly-2U-Hotswap; symbol keyboard_parts:KEYSW -> discipline-pcb-rescue:KEYSW-keyboard_parts
- SW16, SW29: footprint cftkb:SW_Cherry_MX1A_1.50u_PCBNOSCREEN -> MX_Only:MXOnly-1.5U-Hotswap; symbol keyboard_parts:KEYSW -> discipline-pcb-rescue:KEYSW-keyboard_parts
- SW31, SW56: footprint cftkb:SW_Cherry_MX1A_1.75u_PCBNOSCREEN -> MX_Only:MXOnly-1.75U-Hotswap; symbol keyboard_parts:KEYSW -> discipline-pcb-rescue:KEYSW-keyboard_parts
- SW43, SW45: footprint cftkb:SW_Cherry_MX1A_2.25u_PCBNOSCREEN -> MX_Only:MXOnly-2.25U-Hotswap; symbol keyboard_parts:KEYSW -> discipline-pcb-rescue:KEYSW-keyboard_parts
- SW59, SW61, SW63, SW64, SW69: footprint cftkb:SW_Cherry_MX1A_1.25u_PCBNOSCREEN -> MX_Only:MXOnly-1.25U-Hotswap; symbol keyboard_parts:KEYSW -> discipline-pcb-rescue:KEYSW-keyboard_parts
- SW60: footprint cftkb:SW_Cherry_MX1A_1.25u_PCBNOSCREEN -> MX_Only:MXOnly-1U-Hotswap; symbol keyboard_parts:KEYSW -> discipline-pcb-rescue:KEYSW-keyboard_parts
- SW62: footprint cftkb:SW_Cherry_MX1A_1.00u_PCB-NOSCREEN -> MX_Only:MXOnly-7U-Hotswap-ReversedStabilizers; symbol keyboard_parts:KEYSW -> discipline-pcb-rescue:KEYSW-keyboard_parts
- SW70: renamed from SW68; footprint cftkb:SW_Cherry_MX1A_1.00u_PCB-NOSCREEN -> MX_Only:MXOnly-1U-Hotswap; symbol keyboard_parts:KEYSW -> discipline-pcb-rescue:KEYSW-keyboard_parts
- U1: symbol MCU_Microchip_ATmega:ATmega32A-PU -> discipline-pcb-rescue:ATmega32A-PU-MCU_Microchip_ATmega
- USB1: symbol Type-C:USB_C_GCT_USB4085 -> discipline-pcb-rescue:USB_C_GCT_USB4085-Type-C
- renumbered D53 to D10, D54 to D11, D55 to D12, D64 to D13, D57 to D14, D33 to D18, D34 to D19, D35 to D20, D36 to D21, D37 to D22, D38 to D23, D39 to D24, D40 to D25, D41 to D26, D42 to D27, D56 to D28, D46 to D3, D18 to D33, D19 to D34, D20 to D35, D21 to D36, D22 to D37, D23 to D38, D24 to D39, D47 to D4, D25 to D40, D26 to D41, D27 to D42, D28 to D43, D3 to D46, D4 to D47, D5 to D48, D6 to D49, D48 to D5, D7 to D50, D8 to D51, D9 to D52, D10 to D53, D11 to D54, D12 to D55, D13 to D56, D14 to D57, D49 to D6, D68 to D64, D43 to D68, D50 to D7, D51 to D8, D52 to D9
Connections:
- wire segments 342 -> 335
- no-connect marks 9 -> 19
Other:
- moved on the sheet: D10, D11, D12, D13, D14, D18, D19, D20, D21, D22, D23, D24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
