File: discipline-pcb.sch (KiCad schematic (older format))
At the start: 170 parts, among them J1 AVR-ISP-6, SW1 KEYSW, SW10 KEYSW, SW11 KEYSW, SW12 KEYSW, SW13 KEYSW, SW14 KEYSW, SW15 KEYSW, SW16 KEYSW, SW17 KEYSW, SW18 KEYSW, SW19 KEYSW, SW2 KEYSW, SW20 KEYSW, SW21 KEYSW, SW22 KEYSW, SW23 KEYSW, SW24 KEYSW, SW25 KEYSW, SW26 KEYSW, SW27 KEYSW, SW28 KEYSW, SW29 KEYSW, SW3 KEYSW, SW30 KEYSW, SW31 KEYSW, SW32 KEYSW, SW33 KEYSW, SW34 KEYSW, SW35 KEYSW, SW36 KEYSW, SW37 KEYSW, SW38 KEYSW, SW39 KEYSW, SW4 KEYSW, SW40 KEYSW, SW41 KEYSW, SW42 KEYSW, SW43 KEYSW, SW44 KEYSW, SW45 KEYSW, SW46 KEYSW, SW47 KEYSW, SW48 KEYSW, SW49 KEYSW, SW5 KEYSW, SW50 KEYSW, SW51 KEYSW, SW52 KEYSW, SW53 KEYSW, SW54 KEYSW, SW55 KEYSW, SW56 KEYSW, SW57 KEYSW, SW58 KEYSW, SW59 KEYSW, SW6 KEYSW, SW60 KEYSW, SW61 KEYSW, SW62 KEYSW, SW63 KEYSW, SW64 KEYSW, SW65 KEYSW, SW66 KEYSW, SW67 KEYSW, SW68 KEYSW, SW69 KEYSW, SW7 KEYSW, SW70 KEYSW, SW8 KEYSW, SW9 KEYSW, U1 ATmega32A-PU, Y1 Crystal

Commit message: Add alternative bottom row
Parts:
- added SW71: KEYSW, MX_Only:MXOnly-7U-Hotswap, symbol Switch:SW_DIP_x01
- added SW72, SW73, SW75: KEYSW, MX_Only:MXOnly-1.25U-Hotswap, symbol Switch:SW_DIP_x01
- added SW74: KEYSW, MX_Only:MXOnly-1U-Hotswap, symbol Switch:SW_DIP_x01
- BOOT1, RESET1: symbol discipline-pcb-rescue:SW_PUSH-keyboard_parts -> Switch:SW_Push
- C1, C2: footprint cftkb:D_DO-35_SOD27_P5.08mm_Horizontal -> cftkb:C_Disc_D3.0mm_W1.6mm_P2.50mm
- C3: footprint cftkb:D_DO-35_SOD27_P5.08mm_Horizontal -> cftkb:CP_Radial_D4.0mm_P1.50mm
- C4, C5: footprint cftkb:D_DO-35_SOD27_P5.08mm_Horizontal -> cftkb:C_Disc_D4.3mm_W1.9mm_P5.00mm
- J1: symbol discipline-pcb-rescue:AVR-ISP-6-Connector -> Connector:AVR-ISP-6
- SW1, SW10, SW11, SW12, SW13, SW14, SW15, SW16, SW17, SW18, SW19, SW2, SW20, SW21, SW22, SW23, SW24, SW25, SW26, SW27, SW28, SW29, SW3, SW30, SW31, SW32, SW33, SW34, SW35, SW36, SW37, SW38, SW39, SW4, SW40, SW41, SW42, SW43, SW44, SW45, SW46, SW47, SW48, SW49, SW5, SW50, SW51, SW52, SW53, SW54, SW55, SW56, SW57, SW58, SW59, SW6, SW61, SW65, SW66, SW67, SW68, SW69, SW7, SW70, SW8, SW9: symbol discipline-pcb-rescue:KEYSW-keyboard_parts -> Switch:SW_DIP_x01
- SW60: footprint MX_Only:MXOnly-1U-Hotswap -> MX_Only:MXOnly-1.25U-Hotswap; symbol discipline-pcb-rescue:KEYSW-keyboard_parts -> Switch:SW_DIP_x01
- SW62: footprint MX_Only:MXOnly-7U-Hotswap-ReversedStabilizers -> MX_Only:MXOnly-6.25U-Hotswap-ReversedStabilizers; symbol discipline-pcb-rescue:KEYSW-keyboard_parts -> Switch:SW_DIP_x01
- SW63, SW64: footprint MX_Only:MXOnly-1.25U-Hotswap -> MX_Only:MXOnly-1.5U-Hotswap; symbol discipline-pcb-rescue:KEYSW-keyboard_parts -> Switch:SW_DIP_x01
- U1: symbol discipline-pcb-rescue:ATmega32A-PU-MCU_Microchip_ATmega -> MCU_Microchip_ATmega:ATmega32A-PU
- USB1: symbol discipline-pcb-rescue:USB_C_GCT_USB4085-Type-C -> Connector:USB_C_Receptacle_USB2.0
Connections:
- net col1: now also SW74.1
- net col10: now also SW72.1
- net col11: now also SW73.1
- net col2: now also SW75.1
- net col6: now also SW71.1
- net at D60.2 (A), SW60.1: now also SW74.2
- net at D61.2 (A), SW61.1: now also SW75.2
- net at D62.2 (A), SW62.1: now also SW71.2
- net at D63.2 (A), SW63.1: now also SW72.2
- net at D64.2 (A), SW64.1: now also SW73.2
Other:
- moved on the sheet: BOOT1, C1, C2, C3, C4, C5, D69, D70, F1, J1, LED1, R1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
