File: bottom/discipline-pcb.kicad_pcb (KiCad board)
At the start: 2 copper layers, 304.9 x 122.8 mm, 15 parts

Commit message: Add alternative bottom row
Parts:
- removed the G*** at (128.2, 133.8) (x2)
- H1, H10, H2, H3, H4, H5, H6, H7, H8: renamed from REF**; value MountingHole_2.2mm_M2_Pad -> MountingHole_Pad; footprint MountingHole:MountingHole_2.2mm_M2_Pad -> MountingHole:MountingHole_2.2mm_M2_Pad_Via
- H11, H12: renamed from REF**; value MountingHole_4.3mm_M4_Pad -> MountingHole_Pad; footprint MountingHole:MountingHole_4.3mm_M4_Pad -> MountingHole:MountingHole_4.3mm_M4_Pad_Via
- H9: renamed from H1; footprint MountingHole:MountingHole_2.2mm_M2_Pad -> MountingHole:MountingHole_2.2mm_M2_Pad_Via
Connections:
- H1 pad 1: (no net) -> GND
- H10 pad 1: (no net) -> GND
- H11 pad 1: (no net) -> GND
- H12 pad 1: (no net) -> GND
- H2 pad 1: (no net) -> GND
- H3 pad 1: (no net) -> GND
- H4 pad 1: (no net) -> GND
- H5 pad 1: (no net) -> GND
- H6 pad 1: (no net) -> GND
- H7 pad 1: (no net) -> GND
- H8 pad 1: (no net) -> GND
Routing:
- added copper zone on B.Cu, net (none)
- added copper zone on F.Cu, net (none)
- removed copper zone on B.Cu, net GND
- removed copper zone on F.Cu, net GND
Other:
- board text added: "DISCIPLINE - HS"
- board text removed: "coseyfannitutti"
